Commit message: Add initial script for generating proto

File: protos/robot/nugus/robot.urdf (robot description, URDF)
Before this commit: robot onshape, 25 links, 24 joints
Joints:
- removed joint left_knee
- removed joint right_knee
- added joint left_knee_pitch: type revolute, parent left_upper_leg, child left_lower_leg, origin xyz=0.206046 0.0569501 -1.44745e-14 rpy=-4.42146e-14 -3.94129e-15 -1.40554e-13, axis 0 0 1, limit lower=-3.14159 upper=3.14159 effort=1 velocity=20
- added joint right_knee_pitch: type revolute, parent right_upper_leg, child right_lower_leg, origin xyz=0.206046 0.0569501 -7.16788e-15 rpy=-7.0209e-15 3.9968e-14 -5.66214e-15, axis 0 0 1, limit lower=-3.14159 upper=3.14159 effort=1 velocity=20

Commit message: Revert "Add initial script for generating proto"
This reverts commit d084133c0dea69ade8f2869d17aa2ccc42dffd5b.

File: protos/robot/nugus/robot.urdf (robot description, URDF)
Before this commit: robot onshape, 25 links, 24 joints
Joints:
- removed joint left_knee_pitch
- removed joint right_knee_pitch
- added joint left_knee: type revolute, parent left_upper_leg, child left_lower_leg, origin xyz=0.206046 0.0569501 -1.44745e-14 rpy=-4.42146e-14 -3.94129e-15 -1.40554e-13, axis 0 0 1, limit lower=-3.14159 upper=3.14159 effort=1 velocity=20
- added joint right_knee: type revolute, parent right_upper_leg, child right_lower_leg, origin xyz=0.206046 0.0569501 -7.16788e-15 rpy=-7.0209e-15 3.9968e-14 -5.66214e-15, axis 0 0 1, limit lower=-3.14159 upper=3.14159 effort=1 velocity=20

Commit message: Add jersey with colours

File: protos/robot/nugus/robot.urdf (robot description, URDF)
Before this commit: robot onshape, 25 links, 24 joints
Links:
- link head: geometry collision box size=0.16223767679184675 0.15564338862895966 0.15779687464237213; visual mesh filename=head_visual.stl
- link left_lower_arm: geometry collision box size=0.08257202059030533 0.25829844921827316 0.050921617075800896; visual mesh filename=left_lower_arm_visual.stl
- link right_lower_arm: geometry collision box size=0.08257202059030533 0.2583179399371147 0.050956809893250465; visual mesh filename=right_lower_arm_visual.stl
- link right_upper_arm: geometry collision box size=0.22482992708683014 0.07902275025844574 0.08959516510367393; visual mesh filename=right_upper_arm_visual.stl
- link torso: geometry collision box size=0.13950913399457932 0.1899828165769577 0.2618043217808008; visual mesh filename=torso_visual.stl
